Commit message: Cambio a piezas colores simulacion

File: ow_peque_description/urdf/materials.xacro (robot description, xacro)
@@ -13,3 +13,9 @@
             <color rgba="0.5 0 0 1"/>
         </material>
+        <material name="orange">
+            <color rgba="1.0 0.5 0.0 1"/>
+        </material>
+        <material name="black">
+            <color rgba="0.1 0.1 0.1 1"/>
+        </material>
 </robot>

File: ow_peque_description/urdf/mobile_base.xacro (robot description, xacro)
@@ -9,21 +9,50 @@
         <visual>
             <geometry>
-                <mesh filename="file://$(find ow_peque_description)/meshes/EnsamblajeRobotPeque.stl" scale="0.001 0.001 0.001"/>
+                <mesh filename="file://$(find ow_peque_description)/meshes/PiezasNaranjas.stl" scale="0.001 0.001 0.001"/>
             </geometry>
             <origin xyz="0 0 ${base_to_ground_height}" rpy="${pi / 2.0} 0 ${-2.0 * pi / 3.0}"/>
-            <material name="blue"/>
+            <material name="orange"/>
         </visual>
         <collision>
             <geometry>
-                <mesh filename="file://$(find ow_peque_description)/meshes/EnsamblajeRobotPeque.stl" scale="0.001 0.001 0.001"/>
-                <!--cylinder radius="${base_radius}" length="${corner_height - corner_shaft_height }"/-->
+                <mesh filename="file://$(find ow_peque_description)/meshes/ModeloColision.stl" scale="0.001 0.001 0.001"/>
             </geometry>
             <origin xyz="0 0 ${base_to_ground_height}" rpy="${pi / 2.0} 0 ${-2.0 * pi / 3.0}"/>
         </collision>
-         <inertial>
+        <inertial>
             <mass value="5"/>
             <origin xyz="0 0 0" rpy="0 0 0"/>
             <inertia ixx="0.0004055" ixy="0" ixz="0" iyy="0.0004055" iyz="0" izz="0"/>
         </inertial>
+    </link>
+    <!-- Piezas negras (visual separado para permitir diferente color) -->
+    <joint name="base_to_black_parts" type="fixed">
+        <parent link="base_link"/>
+        <child link="black_parts_link"/>
+        <origin xyz="0 0 0" rpy="0 0 0"/>
+    </joint>
+    <link name="black_parts_link">
+        <visual>
+            <geometry>
+                <mesh filename="file://$(find ow_peque_description)/meshes/PiezasNegras.stl" scale="0.001 0.001 0.001"/>
+            </geometry>
+            <origin xyz="0 0 ${base_to_ground_height}" rpy="${pi / 2.0} 0 ${-2.0 * pi / 3.0}"/>
+            <material name="black"/>
+        </visual>
+    </link>
+    <!-- Placas electrónicas -->
+    <joint name="base_to_placas" type="fixed">
+        <parent link="base_link"/>
+        <child link="placas_link"/>
+        <origin xyz="0 0 0" rpy="0 0 0"/>
+    </joint>
+    <link name="placas_link">
+        <visual>
+            <geometry>
+                <mesh filename="file://$(find ow_peque_description)/meshes/Placas.stl" scale="0.001 0.001 0.001"/>
+            </geometry>
+            <origin xyz="0 0 ${base_to_ground_height}" rpy="${pi / 2.0} 0 ${-2.0 * pi / 3.0}"/>
+            <material name="green"/>
+        </visual>
     </link>
     <!-- Ruedas omnidireccionales -->

File: ow_peque_description/urdf/mobile_base_gazebo.xacro (robot description, xacro)
@@ -1,27 +1,30 @@
 <?xml version="1.0"?>
 <robot xmlns:xacro="http://www.ros.org/wiki/xacro">
+    <!-- Base link - Piezas naranjas -->
     <gazebo reference="base_link">
         <visual>
             <material>
-                <ambient>0.0 0.0 1.0 1.0</ambient>
-                <diffuse>0.0 0.0 1.0 1.0</diffuse>
+                <ambient>1.0 0.5 0.0 1.0</ambient>
+                <diffuse>1.0 0.5 0.0 1.0</diffuse>
                 <specular>0.1 0.1 0.1 1.0</specular>
             </material>
         </visual>
     </gazebo>
-    <gazebo reference="bottom_cover_link">
+    <!-- Piezas negras -->
+    <gazebo reference="black_parts_link">
         <visual>
             <material>
-                <ambient>1.0 0.0 0.0 1.0</ambient>
-                <diffuse>1.0 0.0 0.0 1.0</diffuse>
+                <ambient>0.1 0.1 0.1 1.0</ambient>
+                <diffuse>0.1 0.1 0.1 1.0</diffuse>
                 <specular>0.1 0.1 0.1 1.0</specular>
             </material>
         </visual>
     </gazebo>
-    <gazebo reference="top_cover_link">
+    <!-- Placas electrónicas - verde -->
+    <gazebo reference="placas_link">
         <visual>
             <material>
-                <ambient>1.0 0.0 0.0 1.0</ambient>
-                <diffuse>1.0 0.0 0.0 1.0</diffuse>
+                <ambient>0.0 0.5 0.0 1.0</ambient>
+                <diffuse>0.0 0.5 0.0 1.0</diffuse>
                 <specular>0.1 0.1 0.1 1.0</specular>
             </material>
