Commit message: Arreglada orientacion ruedas

File: ow_peque_description/urdf/mobile_base.xacro (robot description, xacro)
@@ -11,5 +11,5 @@
                 <mesh filename="file://$(find ow_peque_description)/meshes/PiezasNaranjas.stl" scale="0.001 0.001 0.001"/>
             </geometry>
-            <origin xyz="0 0 ${base_to_ground_height}" rpy="${pi / 2.0} 0 ${-2.0 * pi / 3.0}"/>
+            <origin xyz="0 0 ${base_to_ground_height}" rpy="${pi / 2.0} 0 ${-2.0 * pi / 3.0 - pi / 2.0}"/>
             <material name="orange"/>
         </visual>
@@ -18,5 +18,5 @@
                 <mesh filename="file://$(find ow_peque_description)/meshes/ModeloColision.stl" scale="0.001 0.001 0.001"/>
             </geometry>
-            <origin xyz="0 0 ${base_to_ground_height}" rpy="${pi / 2.0} 0 ${-2.0 * pi / 3.0}"/>
+            <origin xyz="0 0 ${base_to_ground_height}" rpy="${pi / 2.0} 0 ${-2.0 * pi / 3.0 - pi / 2.0}"/>
         </collision>
         <inertial>
@@ -37,5 +37,5 @@
                 <mesh filename="file://$(find ow_peque_description)/meshes/PiezasNegras.stl" scale="0.001 0.001 0.001"/>
             </geometry>
-            <origin xyz="0 0 ${base_to_ground_height}" rpy="${pi / 2.0} 0 ${-2.0 * pi / 3.0}"/>
+            <origin xyz="0 0 ${base_to_ground_height}" rpy="${pi / 2.0} 0 ${-2.0 * pi / 3.0 - pi / 2.0}"/>
             <material name="black"/>
         </visual>
@@ -52,5 +52,5 @@
                 <mesh filename="file://$(find ow_peque_description)/meshes/Placas.stl" scale="0.001 0.001 0.001"/>
             </geometry>
-            <origin xyz="0 0 ${base_to_ground_height}" rpy="${pi / 2.0} 0 ${-2.0 * pi / 3.0}"/>
+            <origin xyz="0 0 ${base_to_ground_height}" rpy="${pi / 2.0} 0 ${-2.0 * pi / 3.0 - pi / 2.0}"/>
             <material name="green"/>
         </visual>
@@ -62,15 +62,15 @@
                      base_radius="${base_radius}"
                      z_offset="${ground_to_shaft_height}"
-                     angle="${pi / 2.0}"/>
+                     angle="${0}"/>
     <xacro:omniwheel parent_link="base_link"
                      prefix="left"
                      base_radius="${base_radius}"
                      z_offset="${ground_to_shaft_height}"
-                     angle="${pi + pi / 6.0}"/>
+                     angle="${pi + pi / 6.0 - pi / 2.0}"/>
     <xacro:omniwheel parent_link="base_link"
                      prefix="right"
                      base_radius="${base_radius}"
                      z_offset="${ground_to_shaft_height}"
-                     angle="${- pi / 6.0}"/>
+                     angle="${- pi / 6.0 - pi / 2.0}"/>
     <!-- Joints -->
     <joint name="base_joint" type="fixed">

File: ow_peque_description/urdf/mobile_base_gazebo.xacro (robot description, xacro)
@@ -41,5 +41,5 @@
         <mu1>${coef1}</mu1>
         <mu2>${coef2}</mu2>
-        <fdir1>${cos(pi/6.0)} ${-sin(pi/6.0)} 0</fdir1>
+        <fdir1>1.0 0.0 0.0</fdir1>
     </gazebo>
     <gazebo reference="left_wheel_link">
@@ -53,5 +53,5 @@
         <mu1>${coef1}</mu1>
         <mu2>${coef2}</mu2>
-        <fdir1>${-cos(pi/6.0)} ${-sin(pi/6.0)} 0</fdir1>
+        <fdir1>1.0 0.0 0.0</fdir1>
     </gazebo>
     <gazebo reference="front_wheel_link">
@@ -65,5 +65,5 @@
         <mu1>${coef1}</mu1>
         <mu2>${coef2}</mu2>
-        <fdir1>0 1.0 0</fdir1>
+        <fdir1>1.0 0.0 0.0</fdir1>
     </gazebo>
 </robot>

File: ow_peque_description/urdf/ow.urdf.xacro (robot description, xacro)
@@ -2,4 +2,6 @@
 <robot name="ow" xmlns:xacro="http://www.ros.org/wiki/xacro">
     <xacro:arg name="sim_mode" default="true"/>
+    <xacro:arg name="sim_namespace" default="/"/>
+    <xacro:arg name="controller_config" default="controllers.yaml"/>
     <xacro:include filename="common_properties.xacro"/>
     <xacro:include filename="materials.xacro"/>

File: ow_peque_description/urdf/ros2_control.xacro (robot description, xacro)
@@ -34,7 +34,7 @@
         <plugin name="gz_ros2_control::GazeboSimROS2ControlPlugin" filename="libgz_ros2_control-system.so">
             <ros>
-                <namespace>/</namespace>
+                <namespace>$(arg sim_namespace)</namespace>
             </ros>
-            <parameters>$(find ow_peque_description)/config/controllers.yaml</parameters>
+            <parameters>$(find ow_peque_description)/config/$(arg controller_config)</parameters>
             <parameters>$(find ow_peque_description)/config/gaz_ros2_ctl_use_sim.yaml</parameters>
         </plugin>
