Commit message: Cambios para adaptar a la geometria de OW_PEQUE

File: ow_peque_description/urdf/common_properties.xacro (robot description, xacro)
@@ -2,9 +2,9 @@
 <robot xmlns:xacro="http://www.ros.org/wiki/xacro">
     <!--Parametros-->
-    <xacro:property name="base_plate_height" value="0.004"/>
-    <xacro:property name="corner_height" value="0.091"/>
-    <xacro:property name="corner_shaft_height" value="0.04"/>
-    <xacro:property name="omniwheel_radius" value="0.05"/>
-    <xacro:property name="base_radius" value="0.22"/>
+    <xacro:property name="base_plate_height" value="0.018"/>
+    <xacro:property name="base_to_ground_height" value="0.02"/>
+    <xacro:property name="ground_to_shaft_height" value="0.03"/>
+    <xacro:property name="omniwheel_radius" value="0.025"/>
+    <xacro:property name="base_radius" value="0.09"/>
     <!-- Simulación -->
     <xacro:property name="coef1" value="0.5"/>

File: ow_peque_description/urdf/mobile_base.xacro (robot description, xacro)
@@ -9,46 +9,18 @@
         <visual>
             <geometry>
-                <mesh filename="file://$(find ow_description)/meshes/BodyFrame.stl" scale="0.001 0.001 0.001"/>
+                <mesh filename="file://$(find ow_peque_description)/meshes/EnsamblajeRobotPeque.stl" scale="0.001 0.001 0.001"/>
             </geometry>
-            <origin xyz="0 0 ${corner_height - corner_shaft_height }" rpy="0 0 0"/>
+            <origin xyz="0 0 ${base_to_ground_height}" rpy="${pi / 2.0} 0 ${-2.0 * pi / 3.0}"/>
             <material name="blue"/>
         </visual>
         <collision>
             <geometry>
-                <mesh filename="file://$(find ow_description)/meshes/BodyFrame.stl" scale="0.001 0.001 0.001"/>
+                <mesh filename="file://$(find ow_peque_description)/meshes/EnsamblajeRobotPeque.stl" scale="0.001 0.001 0.001"/>
                 <!--cylinder radius="${base_radius}" length="${corner_height - corner_shaft_height }"/-->
             </geometry>
-            <origin xyz="0 0 ${corner_height - corner_shaft_height }" rpy="0 0 0"/>
+            <origin xyz="0 0 ${base_to_ground_height}" rpy="${pi / 2.0} 0 ${-2.0 * pi / 3.0}"/>
         </collision>
          <inertial>
             <mass value="5"/>
-            <origin xyz="0 0 0" rpy="0 0 0"/>
-            <inertia ixx="0.0004055" ixy="0" ixz="0" iyy="0.0004055" iyz="0" izz="0"/>
-        </inertial>
-    </link>
-    <link name="bottom_cover_link">
-        <visual>
-            <geometry>
-                <mesh filename="file://$(find ow_description)/meshes/base.stl" scale="0.001 0.001 0.001"/>
-            </geometry>
-            <origin xyz="0 0 0" rpy="0 0 0"/>
-            <material name="red"/>
-        </visual>
-        <inertial>
-            <mass value="0.129"/>
-            <origin xyz="0 0 0" rpy="0 0 0"/>
-            <inertia ixx="0.0004055" ixy="0" ixz="0" iyy="0.0004055" iyz="0" izz="0"/>
-        </inertial>
-    </link>
-    <link name="top_cover_link">
-        <visual>
-            <geometry>
-                <mesh filename="file://$(find ow_description)/meshes/base.stl" scale="0.001 0.001 0.001"/>
-            </geometry>
-            <origin xyz="0 0 0" rpy="0 0 0"/>
-            <material name="red"/>
-        </visual>
-        <inertial>
-            <mass value="0.129"/>
             <origin xyz="0 0 0" rpy="0 0 0"/>
             <inertia ixx="0.0004055" ixy="0" ixz="0" iyy="0.0004055" iyz="0" izz="0"/>
@@ -59,7 +31,7 @@
             <visual>
                 <geometry>
-                    <mesh filename="file://$(find ow_description)/meshes/omniwheel.stl" scale="0.001 0.001 0.001"/>
+                    <mesh filename="file://$(find ow_peque_description)/meshes/RuedaOmnidireccional.stl" scale="0.001 0.001 0.001"/>
                 </geometry>
-                <origin xyz="0 0 0" rpy="${pi / 2.0} 0 0"/>
+                <origin xyz="0 0 0" rpy="0 0 ${pi / 2.0}"/>
                 <material name="grey"/>
             </visual>
@@ -71,6 +43,6 @@
             <collision>
                 <geometry>
-                    <!--mesh filename="file://$(find ow_description)/meshes/omniwheel.stl" scale="0.001 0.001 0.001"/-->
-                    <cylinder radius="${omniwheel_radius}" length="0.005"/>
+                    <!--mesh filename="file://$(find ow_peque_description)/meshes/omniwheel.stl" scale="0.001 0.001 0.001"/-->
+                    <cylinder radius="${omniwheel_radius}" length="0.02"/>
                 </geometry>
                 <origin xyz="0 0 0" rpy="${pi / 2.0} 0 0"/>
@@ -80,5 +52,8 @@
             <parent link="base_link"/>
             <child link="${prefix}_wheel_link"/>
-            <origin xyz="${cos (angle) * base_radius} ${sin (angle) * base_radius} 0" rpy="0 0 ${angle - pi / 2.0}"/>
+            <!-- Use 0 for the wheel joint z origin to match the other description
+                 and avoid a 0 -> 0.05 jump in RViz when multiple descriptions
+                 or TF sources are present. -->
+            <origin xyz="${cos (angle) * base_radius} ${sin (angle) * base_radius} ${ground_to_shaft_height}" rpy="0 0 ${angle - pi / 2.0}"/>
             <axis xyz="0 1 0"/>
         </joint>
@@ -93,13 +68,3 @@
         <origin xyz="0 0 ${omniwheel_radius}" rpy="0 0 0"/>
     </joint>
-    <joint name="base_bottom_cover_joint" type="fixed">
-        <parent link="base_link"/>
-        <child link="bottom_cover_link"/>
-        <origin xyz="0 0 ${-corner_shaft_height + base_plate_height * 2 }" rpy="0 0 0"/>
-    </joint>
-    <joint name="base_top_cover_joint" type="fixed">
-        <parent link="base_link"/>
-        <child link="top_cover_link"/>
-        <origin xyz="0 0 ${corner_height - corner_shaft_height }" rpy="0 0 0"/>
-    </joint>
 </robot>

File: ow_peque_description/urdf/omniwheel.xacro (robot description, xacro)
@@ -4,5 +4,5 @@
     <visual>
       <geometry>
-        <mesh filename="file://$(find ow_description)/meshes/OmniwheelBody.stl" scale="0.001 0.001 0.001"/>
+        <mesh filename="file://$(find ow_peque_description)/meshes/RuedaOmnidireccional.stl" scale="0.001 0.001 0.001"/>
       </geometry>
       <origin xyz="0 0 0" rpy="0 0 0"/>

File: ow_peque_description/urdf/ow.urdf.xacro (robot description, xacro)
@@ -3,8 +3,4 @@
     <xacro:include filename="common_properties.xacro"/>
     <xacro:include filename="materials.xacro"/>
-    <!-- Plugin de ros2_control para manejar el robot-->
-    <xacro:include filename="ros2_control.xacro"/>
     <xacro:include filename="mobile_base.xacro"/>
-    <xacro:include filename="mobile_base_gazebo.xacro"/>
-    <!--xacro:include filename="omniwheel.xacro"/-->
 </robot>

Commit message: Movemos la rueda omnidireccional a su propio archivo

File: ow_peque_description/urdf/common_properties.xacro (robot description, xacro)
@@ -5,5 +5,5 @@
     <xacro:property name="base_to_ground_height" value="0.02"/>
     <xacro:property name="ground_to_shaft_height" value="0.03"/>
-    <xacro:property name="omniwheel_radius" value="0.025"/>
+    <xacro:property name="omniwheel_radius" value="0.029"/>
     <xacro:property name="base_radius" value="0.09"/>
     <!-- Simulación -->

File: ow_peque_description/urdf/mobile_base.xacro (robot description, xacro)
@@ -27,39 +27,21 @@
         </inertial>
     </link>
-    <xacro:macro name="omniwheel" params="prefix angle">
-        <link name="${prefix}_wheel_link">
-            <visual>
-                <geometry>
-                    <mesh filename="file://$(find ow_peque_description)/meshes/RuedaOmnidireccional.stl" scale="0.001 0.001 0.001"/>
-                </geometry>
-                <origin xyz="0 0 0" rpy="0 0 ${pi / 2.0}"/>
-                <material name="grey"/>
-            </visual>
-            <inertial>
-                <mass value="0.582"/>
-                <origin xyz="0 0 0" rpy="0 0 0"/>
-                <inertia ixx="0.0005937" ixy="0" ixz="0" iyy="0.0005937" iyz="0" izz="0.0009841"/>
-            </inertial>
-            <collision>
-                <geometry>
-                    <!--mesh filename="file://$(find ow_peque_description)/meshes/omniwheel.stl" scale="0.001 0.001 0.001"/-->
-                    <cylinder radius="${omniwheel_radius}" length="0.02"/>
-                </geometry>
-                <origin xyz="0 0 0" rpy="${pi / 2.0} 0 0"/>
-            </collision>
-        </link>
-        <joint name="base_${prefix}_wheel_joint" type="continuous">
-            <parent link="base_link"/>
-            <child link="${prefix}_wheel_link"/>
-            <!-- Use 0 for the wheel joint z origin to match the other description
-                 and avoid a 0 -> 0.05 jump in RViz when multiple descriptions
-                 or TF sources are present. -->
-            <origin xyz="${cos (angle) * base_radius} ${sin (angle) * base_radius} ${ground_to_shaft_height}" rpy="0 0 ${angle - pi / 2.0}"/>
-            <axis xyz="0 1 0"/>
-        </joint>
-    </xacro:macro>
-    <xacro:omniwheel prefix="front" angle="${pi / 2.0}"/>
-    <xacro:omniwheel prefix="left" angle="${pi + pi / 6.0}"/>
-    <xacro:omniwheel prefix="right" angle="${- pi / 6.0}"/>
+    <!-- Ruedas omnidireccionales -->
+    <xacro:include filename="$(find ow_peque_description)/urdf/omniwheel.xacro"/>
+    <xacro:omniwheel parent_link="base_link"
+                     prefix="front"
+                     base_radius="${base_radius}"
+                     z_offset="${ground_to_shaft_height}"
+                     angle="${pi / 2.0}"/>
+    <xacro:omniwheel parent_link="base_link"
+                     prefix="left"
+                     base_radius="${base_radius}"
+                     z_offset="${ground_to_shaft_height}"
+                     angle="${pi + pi / 6.0}"/>
+    <xacro:omniwheel parent_link="base_link"
+                     prefix="right"
+                     base_radius="${base_radius}"
+                     z_offset="${ground_to_shaft_height}"
+                     angle="${- pi / 6.0}"/>
     <!-- Joints -->
     <joint name="base_joint" type="fixed">

File: ow_peque_description/urdf/omniwheel.xacro (robot description, xacro)
@@ -1,17 +1,32 @@
 <?xml version="1.0"?>
 <robot xmlns:xacro="http://www.ros.org/wiki/xacro">
-  <link name="omniwheel_link">
-    <visual>
-      <geometry>
-        <mesh filename="file://$(find ow_peque_description)/meshes/RuedaOmnidireccional.stl" scale="0.001 0.001 0.001"/>
-      </geometry>
-      <origin xyz="0 0 0" rpy="0 0 0"/>
-    </visual>
-  </link>
-  <joint name="omniwheel_joint" type="continuous">
-    <parent link="base_link"/>
-    <child link="omniwheel_link"/>
-    <origin xyz="0 0 0" rpy="0 0 0"/>
-    <axis xyz="0 0 1"/>
-  </joint>
+  <xacro:macro name="omniwheel" params="parent_link prefix angle base_radius z_offset">
+        <link name="${prefix}_wheel_link">
+            <visual>
+                <geometry>
+                    <mesh filename="file://$(find ow_peque_description)/meshes/RuedaOmnidireccional.stl" scale="0.001 0.001 0.001"/>
+                </geometry>
+                <origin xyz="0 0 0" rpy="0 0 ${pi / 2.0}"/>
+                <material name="grey"/>
+            </visual>
+            <inertial>
+                <mass value="0.582"/>
+                <origin xyz="0 0 0" rpy="0 0 0"/>
+                <inertia ixx="0.0005937" ixy="0" ixz="0" iyy="0.0005937" iyz="0" izz="0.0009841"/>
+            </inertial>
+            <collision>
+                <geometry>
+                    <!-- Para que sea más sencilla la simulación, se usa una geometría cilíndrica en lugar de la malla -->
+                    <cylinder radius="0.029" length="0.02"/>
+                </geometry>
+                <origin xyz="0 0 0" rpy="${pi / 2.0} 0 0"/>
+            </collision>
+        </link>
+        <joint name="base_${prefix}_wheel_joint" type="continuous">
+            <parent link="${parent_link}"/>
+            <child link="${prefix}_wheel_link"/>
+            <origin xyz="${cos (angle) * base_radius} ${sin (angle) * base_radius} ${z_offset}" rpy="0 0 ${angle - pi / 2.0}"/>
+            <axis xyz="0 1 0"/>
+        </joint>
+    </xacro:macro>
 </robot>

File: ow_peque_description/urdf/ow.urdf.xacro (robot description, xacro)
@@ -1,4 +1,6 @@
 <?xml version="1.0"?>
 <robot name="ow" xmlns:xacro="http://www.ros.org/wiki/xacro">
+    <xacro:arg name="use_ros2_control" default="true"/>
+    <xacro:arg name="sim_mode" default="false"/>
     <xacro:include filename="common_properties.xacro"/>
     <xacro:include filename="materials.xacro"/>

Commit message: Adaptacion coeficientes y colores a nuevo gazebo

File: ow_peque_description/urdf/common_properties.xacro (robot description, xacro)
@@ -8,5 +8,5 @@
     <xacro:property name="base_radius" value="0.09"/>
     <!-- Simulación -->
-    <xacro:property name="coef1" value="0.5"/>
-    <xacro:property name="coef2" value="0.5"/>
+    <xacro:property name="coef1" value="1.0"/>
+    <xacro:property name="coef2" value="0.001"/>
 </robot>

File: ow_peque_description/urdf/mobile_base_gazebo.xacro (robot description, xacro)
@@ -2,27 +2,63 @@
 <robot xmlns:xacro="http://www.ros.org/wiki/xacro">
     <gazebo reference="base_link">
-        <material>Gazebo/Blue</material>
+        <visual>
+            <material>
+                <ambient>0.0 0.0 1.0 1.0</ambient>
+                <diffuse>0.0 0.0 1.0 1.0</diffuse>
+                <specular>0.1 0.1 0.1 1.0</specular>
+            </material>
+        </visual>
     </gazebo>
     <gazebo reference="bottom_cover_link">
-        <material>Gazebo/Red</material>
+        <visual>
+            <material>
+                <ambient>1.0 0.0 0.0 1.0</ambient>
+                <diffuse>1.0 0.0 0.0 1.0</diffuse>
+                <specular>0.1 0.1 0.1 1.0</specular>
+            </material>
+        </visual>
     </gazebo>
     <gazebo reference="top_cover_link">
-        <material>Gazebo/Red</material>
+        <visual>
+            <material>
+                <ambient>1.0 0.0 0.0 1.0</ambient>
+                <diffuse>1.0 0.0 0.0 1.0</diffuse>
+                <specular>0.1 0.1 0.1 1.0</specular>
+            </material>
+        </visual>
     </gazebo>
     <gazebo reference="right_wheel_link">
-        <material>Gazebo/Grey</material>
-        <mu>${coef1}</mu>
+        <visual>
+            <material>
+                <ambient>0.5 0.5 0.5 1.0</ambient>
+                <diffuse>0.5 0.5 0.5 1.0</diffuse>
+                <specular>0.1 0.1 0.1 1.0</specular>
+            </material>
+        </visual>
+        <mu1>${coef1}</mu1>
         <mu2>${coef2}</mu2>
         <fdir1>${cos(pi/6.0)} ${-sin(pi/6.0)} 0</fdir1>
     </gazebo>
     <gazebo reference="left_wheel_link">
-        <material>Gazebo/Grey</material>
-        <mu>${coef1}</mu>
+        <visual>
+            <material>
+                <ambient>0.5 0.5 0.5 1.0</ambient>
+                <diffuse>0.5 0.5 0.5 1.0</diffuse>
+                <specular>0.1 0.1 0.1 1.0</specular>
+            </material>
+        </visual>
+        <mu1>${coef1}</mu1>
         <mu2>${coef2}</mu2>
         <fdir1>${-cos(pi/6.0)} ${-sin(pi/6.0)} 0</fdir1>
     </gazebo>
     <gazebo reference="front_wheel_link">
-        <material>Gazebo/Grey</material>
-        <mu>${coef1}</mu>
+        <visual>
+            <material>
+                <ambient>0.5 0.5 0.5 1.0</ambient>
+                <diffuse>0.5 0.5 0.5 1.0</diffuse>
+                <specular>0.1 0.1 0.1 1.0</specular>
+            </material>
+        </visual>
+        <mu1>${coef1}</mu1>
         <mu2>${coef2}</mu2>
         <fdir1>0 1.0 0</fdir1>

Commit message: ow_peque_description: calibrar robot_radius a 0.083 m
Ajustado robot_radius de 0.09 a 0.083 m tras medición física
del robot. Corrige el drift acumulado en rotación del dead reckoning.

File: ow_peque_description/urdf/common_properties.xacro (robot description, xacro)
@@ -6,5 +6,5 @@
     <xacro:property name="ground_to_shaft_height" value="0.03"/>
     <xacro:property name="omniwheel_radius" value="0.029"/>
-    <xacro:property name="base_radius" value="0.09"/>
+    <xacro:property name="base_radius" value="0.083"/>
     <!-- Simulación -->
     <xacro:property name="coef1" value="1.0"/>

Commit message: Cambio medida distancia ruedas experimental

File: ow_peque_description/urdf/common_properties.xacro (robot description, xacro)
@@ -6,5 +6,5 @@
     <xacro:property name="ground_to_shaft_height" value="0.03"/>
     <xacro:property name="omniwheel_radius" value="0.029"/>
-    <xacro:property name="base_radius" value="0.083"/>
+    <xacro:property name="base_radius" value="0.095"/>
     <!-- Simulación -->
     <xacro:property name="coef1" value="1.0"/>

Commit message: Pruebas experimentales de ruedas

File: ow_peque_description/urdf/common_properties.xacro (robot description, xacro)
@@ -6,5 +6,5 @@
     <xacro:property name="ground_to_shaft_height" value="0.03"/>
     <xacro:property name="omniwheel_radius" value="0.029"/>
-    <xacro:property name="base_radius" value="0.095"/>
+    <xacro:property name="base_radius" value="0.0937"/>
     <!-- Simulación -->
     <xacro:property name="coef1" value="1.0"/>

Commit message: Otro valor de prueba

File: ow_peque_description/urdf/common_properties.xacro (robot description, xacro)
@@ -6,5 +6,5 @@
     <xacro:property name="ground_to_shaft_height" value="0.03"/>
     <xacro:property name="omniwheel_radius" value="0.029"/>
-    <xacro:property name="base_radius" value="0.0937"/>
+    <xacro:property name="base_radius" value="0.0934"/>
     <!-- Simulación -->
     <xacro:property name="coef1" value="1.0"/>

Commit message: Prueba distancia, diminuimos wheel_radius

File: ow_peque_description/urdf/common_properties.xacro (robot description, xacro)
@@ -5,5 +5,5 @@
     <xacro:property name="base_to_ground_height" value="0.02"/>
     <xacro:property name="ground_to_shaft_height" value="0.03"/>
-    <xacro:property name="omniwheel_radius" value="0.029"/>
+    <xacro:property name="omniwheel_radius" value="0.0294"/>
     <xacro:property name="base_radius" value="0.0934"/>
     <!-- Simulación -->

Commit message: Prueba distancia 2, diminuimos wheel_radius

File: ow_peque_description/urdf/common_properties.xacro (robot description, xacro)
@@ -5,5 +5,5 @@
     <xacro:property name="base_to_ground_height" value="0.02"/>
     <xacro:property name="ground_to_shaft_height" value="0.03"/>
-    <xacro:property name="omniwheel_radius" value="0.0294"/>
+    <xacro:property name="omniwheel_radius" value="0.0288"/>
     <xacro:property name="base_radius" value="0.0934"/>
     <!-- Simulación -->

Commit message: Prueba distancia 3, aumentamos wheel_radius

File: ow_peque_description/urdf/common_properties.xacro (robot description, xacro)
@@ -5,5 +5,5 @@
     <xacro:property name="base_to_ground_height" value="0.02"/>
     <xacro:property name="ground_to_shaft_height" value="0.03"/>
-    <xacro:property name="omniwheel_radius" value="0.0288"/>
+    <xacro:property name="omniwheel_radius" value="0.0300"/>
     <xacro:property name="base_radius" value="0.0934"/>
     <!-- Simulación -->

Commit message: Prueba distancia 4, disminuimos wheel_radius

File: ow_peque_description/urdf/common_properties.xacro (robot description, xacro)
@@ -5,5 +5,5 @@
     <xacro:property name="base_to_ground_height" value="0.02"/>
     <xacro:property name="ground_to_shaft_height" value="0.03"/>
-    <xacro:property name="omniwheel_radius" value="0.0300"/>
+    <xacro:property name="omniwheel_radius" value="0.029"/>
     <xacro:property name="base_radius" value="0.0934"/>
     <!-- Simulación -->

Commit message: Calibrado teniendo en cuenta el ratio

File: ow_peque_description/urdf/common_properties.xacro (robot description, xacro)
@@ -6,5 +6,5 @@
     <xacro:property name="ground_to_shaft_height" value="0.03"/>
     <xacro:property name="omniwheel_radius" value="0.029"/>
-    <xacro:property name="base_radius" value="0.0934"/>
+    <xacro:property name="base_radius" value="0.0821"/>
     <!-- Simulación -->
     <xacro:property name="coef1" value="1.0"/>
