Commit message: Implementado control omnidireccional

File: ow_description/urdf/common_properties.xacro (robot description, xacro)
@@ -8,5 +8,5 @@
     <xacro:property name="base_radius" value="0.22"/>
     <!-- Simulación -->
-    <xacro:property name="coef1" value="1"/>
-    <xacro:property name="coef2" value="1"/>
+    <xacro:property name="coef1" value="100"/>
+    <xacro:property name="coef2" value="0.1"/>
 </robot>

Commit message: Funcionando con mando y fricciones corregidas
Se ha incluido el driver del controlador de ps4
Y se ha conseguido arreglar los coeficientes de fricción de las ruedas en gazebo que dependian de la orientacion de la rueda.

File: ow_description/urdf/common_properties.xacro (robot description, xacro)
@@ -8,5 +8,5 @@
     <xacro:property name="base_radius" value="0.22"/>
     <!-- Simulación -->
-    <xacro:property name="coef1" value="100"/>
-    <xacro:property name="coef2" value="0.1"/>
+    <xacro:property name="coef1" value="0.5"/>
+    <xacro:property name="coef2" value="0.5"/>
 </robot>

File: ow_description/urdf/mobile_base.xacro (robot description, xacro)
@@ -71,5 +71,6 @@
             <collision>
                 <geometry>
-                    <mesh filename="file://$(find ow_description)/meshes/omniwheel.stl" scale="0.001 0.001 0.001"/>
+                    <!--mesh filename="file://$(find ow_description)/meshes/omniwheel.stl" scale="0.001 0.001 0.001"/-->
+                    <cylinder radius="${omniwheel_radius}" length="0.005"/>
                 </geometry>
                 <origin xyz="0 0 0" rpy="${pi / 2.0} 0 0"/>

File: ow_description/urdf/mobile_base_gazebo.xacro (robot description, xacro)
@@ -14,4 +14,5 @@
         <mu>${coef1}</mu>
         <mu2>${coef2}</mu2>
+        <fdir1>${cos(pi/6.0)} ${-sin(pi/6.0)} 0</fdir1>
     </gazebo>
     <gazebo reference="left_wheel_link">
@@ -19,4 +20,5 @@
         <mu>${coef1}</mu>
         <mu2>${coef2}</mu2>
+        <fdir1>${-cos(pi/6.0)} ${-sin(pi/6.0)} 0</fdir1>
     </gazebo>
     <gazebo reference="front_wheel_link">
@@ -24,4 +26,5 @@
         <mu>${coef1}</mu>
         <mu2>${coef2}</mu2>
+        <fdir1>0 1.0 0</fdir1>
     </gazebo>
 </robot>

File: ow_description/urdf/ros2_control.xacro (robot description, xacro)
@@ -7,6 +7,6 @@
         <joint name="base_left_wheel_joint">
             <command_interface name="velocity">
-                <param name="min">-10.0</param>
-                <param name="max">10.0</param>
+                <param name="min">-5.0</param>
+                <param name="max">5.0</param>
             </command_interface>
             <state_interface name="velocity"/>
@@ -15,6 +15,6 @@
         <joint name="base_front_wheel_joint">
             <command_interface name="velocity">
-                <param name="min">-10.0</param>
-                <param name="max">10.0</param>
+                <param name="min">-5.0</param>
+                <param name="max">5.0</param>
             </command_interface>
             <state_interface name="velocity"/>
@@ -23,6 +23,6 @@
         <joint name="base_right_wheel_joint">
             <command_interface name="velocity">
-                <param name="min">-10.0</param>
-                <param name="max">10.0</param>
+                <param name="min">-5.0</param>
+                <param name="max">5.0</param>
             </command_interface>
             <state_interface name="velocity"/>

Commit message: Adaptado ow_description al nuevo gazebo

File: ow_description/urdf/common_properties.xacro (robot description, xacro)
@@ -8,5 +8,5 @@
     <xacro:property name="base_radius" value="0.22"/>
     <!-- Simulación -->
-    <xacro:property name="coef1" value="0.5"/>
-    <xacro:property name="coef2" value="0.5"/>
+    <xacro:property name="coef1" value="1.0"/>
+    <xacro:property name="coef2" value="0.001"/>
 </robot>

File: ow_description/urdf/mobile_base.xacro (robot description, xacro)
@@ -91,5 +91,5 @@
         <parent link="base_footprint"/>
         <child link="base_link"/>
-        <origin xyz="0 0 ${omniwheel_radius}" rpy="0 0 0"/>
+        <origin xyz="0 0 ${omniwheel_radius}" rpy="0 0 ${-pi/2.0}"/>
     </joint>
     <joint name="base_bottom_cover_joint" type="fixed">

File: ow_description/urdf/mobile_base_gazebo.xacro (robot description, xacro)
@@ -1,30 +1,69 @@
 <?xml version="1.0"?>
 <robot xmlns:xacro="http://www.ros.org/wiki/xacro">
+    <!-- Base Link - Blue -->
     <gazebo reference="base_link">
-        <material>Gazebo/Blue</material>
+        <visual>
+            <material>
+                <ambient>0.0 0.0 1.0 1.0</ambient>
+                <diffuse>0.0 0.0 1.0 1.0</diffuse>
+                <specular>0.1 0.1 0.1 1.0</specular>
+            </material>
+        </visual>
     </gazebo>
+    <!-- Covers - Red -->
     <gazebo reference="bottom_cover_link">
-        <material>Gazebo/Red</material>
+        <visual>
+            <material>
+                <ambient>1.0 0.0 0.0 1.0</ambient>
+                <diffuse>1.0 0.0 0.0 1.0</diffuse>
+                <specular>0.1 0.1 0.1 1.0</specular>
+            </material>
+        </visual>
     </gazebo>
     <gazebo reference="top_cover_link">
-        <material>Gazebo/Red</material>
+        <visual>
+            <material>
+                <ambient>1.0 0.0 0.0 1.0</ambient>
+                <diffuse>1.0 0.0 0.0 1.0</diffuse>
+                <specular>0.1 0.1 0.1 1.0</specular>
+            </material>
+        </visual>
     </gazebo>
+    <!-- Wheels - Grey -->
     <gazebo reference="right_wheel_link">
-        <material>Gazebo/Grey</material>
-        <mu>${coef1}</mu>
+        <visual>
+            <material>
+                <ambient>0.5 0.5 0.5 1.0</ambient>
+                <diffuse>0.5 0.5 0.5 1.0</diffuse>
+                <specular>0.1 0.1 0.1 1.0</specular>
+            </material>
+        </visual>
+        <mu1>${coef1}</mu1>
         <mu2>${coef2}</mu2>
-        <fdir1>${cos(pi/6.0)} ${-sin(pi/6.0)} 0</fdir1>
+        <fdir1>1 0 0</fdir1>
     </gazebo>
     <gazebo reference="left_wheel_link">
-        <material>Gazebo/Grey</material>
-        <mu>${coef1}</mu>
+        <visual>
+            <material>
+                <ambient>0.5 0.5 0.5 1.0</ambient>
+                <diffuse>0.5 0.5 0.5 1.0</diffuse>
+                <specular>0.1 0.1 0.1 1.0</specular>
+            </material>
+        </visual>
+        <mu1>${coef1}</mu1>
         <mu2>${coef2}</mu2>
-        <fdir1>${-cos(pi/6.0)} ${-sin(pi/6.0)} 0</fdir1>
+        <fdir1>1 0 0</fdir1>
     </gazebo>
     <gazebo reference="front_wheel_link">
-        <material>Gazebo/Grey</material>
-        <mu>${coef1}</mu>
+        <visual>
+            <material>
+                <ambient>0.5 0.5 0.5 1.0</ambient>
+                <diffuse>0.5 0.5 0.5 1.0</diffuse>
+                <specular>0.1 0.1 0.1 1.0</specular>
+            </material>
+        </visual>
+        <mu1>${coef1}</mu1>
         <mu2>${coef2}</mu2>
-        <fdir1>0 1.0 0</fdir1>
+        <fdir1>1 0 0</fdir1>
     </gazebo>
 </robot>

File: ow_description/urdf/ow.urdf.xacro (robot description, xacro)
@@ -1,4 +1,7 @@
 <?xml version="1.0"?>
 <robot name="ow" xmlns:xacro="http://www.ros.org/wiki/xacro">
+    <xacro:arg name="sim_mode" default="true"/>
+    <xacro:arg name="sim_namespace" default="/"/>
+    <xacro:arg name="controller_config" default="controllers.yaml"/>
     <xacro:include filename="common_properties.xacro"/>
     <xacro:include filename="materials.xacro"/>

File: ow_description/urdf/ros2_control.xacro (robot description, xacro)
@@ -1,37 +1,75 @@
 <?xml version="1.0"?>
 <robot xmlns:xacro="https://www.ros.org/wiki/xacro">
-    <ros2_control name="GazeboSystem" type="system">
-        <hardware>
-            <plugin>gazebo_ros2_control/GazeboSystem</plugin>
-        </hardware>
-        <joint name="base_left_wheel_joint">
-            <command_interface name="velocity">
-                <param name="min">-5.0</param>
-                <param name="max">5.0</param>
-            </command_interface>
-            <state_interface name="velocity"/>
-            <state_interface name="position"/>
-        </joint>
-        <joint name="base_front_wheel_joint">
-            <command_interface name="velocity">
-                <param name="min">-5.0</param>
-                <param name="max">5.0</param>
-            </command_interface>
-            <state_interface name="velocity"/>
-            <state_interface name="position"/>
-        </joint>
-        <joint name="base_right_wheel_joint">
-            <command_interface name="velocity">
-                <param name="min">-5.0</param>
-                <param name="max">5.0</param>
-            </command_interface>
-            <state_interface name="velocity"/>
-            <state_interface name="position"/>
-        </joint>
-    </ros2_control>
-    <gazebo>
-        <plugin name="gazebo_ros2_control" filename="libgazebo_ros2_control.so">
-            <parameters>$(find ow_description)/config/my_controllers.yaml</parameters>
-        </plugin>
-    </gazebo>
+    <xacro:if value="$(arg sim_mode)">
+        <ros2_control name="GazeboSimSystem" type="system">
+            <hardware>
+                <plugin>gz_ros2_control/GazeboSimSystem</plugin>
+            </hardware>
+            <joint name="base_front_wheel_joint">
+                <command_interface name="velocity">
+                    <param name="min">-10.0</param>
+                    <param name="max">10.0</param>
+                </command_interface>
+                <state_interface name="position"/>
+                <state_interface name="velocity"/>
+            </joint>
+            <joint name="base_left_wheel_joint">
+                <command_interface name="velocity">
+                    <param name="min">-10.0</param>
+                    <param name="max">10.0</param>
+                </command_interface>
+                <state_interface name="position"/>
+                <state_interface name="velocity"/>
+            </joint>
+            <joint name="base_right_wheel_joint">
+                <command_interface name="velocity">
+                    <param name="min">-10.0</param>
+                    <param name="max">10.0</param>
+                </command_interface>
+                <state_interface name="position"/>
+                <state_interface name="velocity"/>
+            </joint>
+        </ros2_control>
+        <gazebo>
+            <plugin name="gz_ros2_control::GazeboSimROS2ControlPlugin" filename="libgz_ros2_control-system.so">
+                <ros>
+                    <namespace>$(arg sim_namespace)</namespace>
+                </ros>
+                <parameters>$(find ow_description)/config/$(arg controller_config)</parameters>
+                <parameters>$(find ow_description)/config/gaz_ros2_ctl_use_sim.yaml</parameters>
+            </plugin>
+        </gazebo>
+    </xacro:if>
+    <xacro:unless value="$(arg sim_mode)">
+        <!-- Placeholder for real hardware interface -->
+        <ros2_control name="GazeboSystem" type="system">
+            <hardware>
+                <plugin>gazebo_ros2_control/GazeboSystem</plugin>
+            </hardware>
+             <joint name="base_front_wheel_joint">
+                <command_interface name="velocity">
+                    <param name="min">-5.0</param>
+                    <param name="max">5.0</param>
+                </command_interface>
+                <state_interface name="velocity"/>
+                <state_interface name="position"/>
+            </joint>
+            <joint name="base_left_wheel_joint">
+                <command_interface name="velocity">
+                    <param name="min">-5.0</param>
+                    <param name="max">5.0</param>
+                </command_interface>
+                <state_interface name="velocity"/>
+                <state_interface name="position"/>
+            </joint>
+            <joint name="base_right_wheel_joint">
+                <command_interface name="velocity">
+                    <param name="min">-5.0</param>
+                    <param name="max">5.0</param>
+                </command_interface>
+                <state_interface name="velocity"/>
+                <state_interface name="position"/>
+            </joint>
+        </ros2_control>
+    </xacro:unless>
 </robot>
